Commit message: change modles for crobat v1.5

File: robots/crobat/urdf/full_actuated.urdf.xacro (robot description, xacro)
@@ -23,6 +23,6 @@
     <link name="base_link">
       <inertial>
-        <origin xyz="0.0004 -0.0001 0.13193" rpy="0 0 0"/>
-        <mass value="0.08844"/>
+        <origin xyz="0.0003 -0.0007 0.1399" rpy="0 0 0"/>
+        <mass value="0.0566"/>
         <inertia
             ixx="0.00008943" iyy="0.00008943" izz="0.00006466"
@@ -56,5 +56,5 @@
       <child link="fc"/>
       <parent link="base_link"/>
-      <origin rpy="0 0 0" xyz="-0.01735 0.00115 0.15409"/>
+      <origin rpy="0 0 0" xyz="0.000 0.01575 0.14778"/>
       <axis xyz="0 0 1"/>
     </joint>
@@ -62,6 +62,6 @@
     <link name="rotor_arm${child1}">
       <inertial>
-        <origin xyz="-0.0191 0 0.0058" rpy="0 0 0"/>
-        <mass value="0.01512"/>
+        <origin xyz="-0.0099 0.000 0.0036" rpy="0 0 0"/>
+        <mass value="0.0028"/>
         <inertia
             ixx="0.00000144" ixy="0.0" ixz="0.0"
@@ -85,11 +85,11 @@
       <parent link="base_link"/>
       <child link="rotor_arm${child1}"/>
-     <origin rpy="0 0 ${pi/4}" xyz="0.05677 0.05677 0.11771"/>
+     <origin rpy="0 0 ${pi/4}" xyz="0.04423 0.04417 0.12801"/>
       <axis xyz="0 0 1"/>
     </joint>
     <link name="rotor_arm${child2}">
       <inertial>
-        <origin xyz="-0.0191 0 0.0058" rpy="0 0 0"/>
-        <mass value="0.01512"/>
+        <origin xyz="-0.0099 0.000 0.0036" rpy="0 0 0"/>
+        <mass value="0.0028"/>
         <inertia
             ixx="0.00000144" ixy="0.0" ixz="0.0"
@@ -113,11 +113,11 @@
       <parent link="base_link"/>
       <child link="rotor_arm${child2}"/>
-      <origin rpy="0 0 ${pi*3.0/4.0}" xyz="-0.05677 0.05677 0.11771"/>
+      <origin rpy="0 0 ${pi*3.0/4.0}" xyz="-0.04423 0.04417 0.12801"/>
       <axis xyz="0 0 1"/>
     </joint>
     <link name="rotor_arm${child3}">
       <inertial>
-        <origin xyz="-0.0191 0 0.0058" rpy="0 0 0"/>
-        <mass value="0.01512"/>
+        <origin xyz="-0.0099 0.000 0.0036" rpy="0 0 0"/>
+        <mass value="0.0028"/>
         <inertia
             ixx="0.00000144" ixy="0.0" ixz="0.0"
@@ -141,11 +141,11 @@
       <parent link="base_link"/>
       <child link="rotor_arm${child3}"/>
-      <origin rpy="0 0 ${5*pi/4}" xyz="-0.05677 -0.05677 0.11771"/>
+      <origin rpy="0 0 ${5*pi/4}" xyz="-0.04423 -0.04417 0.12801"/>
       <axis xyz="0 0 1"/>
     </joint>
     <link name="rotor_arm${child4}">
       <inertial>
-        <origin xyz="-0.0191 0 0.0058" rpy="0 0 0"/>
-        <mass value="0.01512"/>
+        <origin xyz="-0.0099 0.000 0.0036" rpy="0 0 0"/>
+        <mass value="0.0028"/>
         <inertia
             ixx="0.00000144" ixy="0.0" ixz="0.0"
@@ -169,5 +169,5 @@
       <parent link="base_link"/>
       <child link="rotor_arm${child4}"/>
-      <origin rpy="0 0 ${-pi/4}" xyz="0.05677 -0.05677 0.11771"/>
+      <origin rpy="0 0 ${-pi/4}" xyz="0.04423 -0.04417 0.12801"/>
       <axis xyz="0 0 1"/>
     </joint>
@@ -179,9 +179,9 @@
     <link name="gimbal_link${self}">
       <inertial>
-        <origin xyz="0.04691 0.00 -0.00138" rpy="0 0 0"/>
+        <origin xyz="0.04652 0.00 0.00168" rpy="0 0 0"/>
         <mass value="0.0286"/>
         <inertia
-            ixx="0.00001392" iyy="0.00009886" izz="0.00008593"
-            ixy="0.0000" ixz="-0.0000" iyz="0.00001994"/>
+            ixx="0.000017" iyy="0.0000941" izz="0.0000798"
+            ixy="0.0000" ixz="-0.0000" iyz="0.0000"/>
       </inertial>
       <collision>
@@ -228,5 +228,5 @@
       <parent link="rotor_arm${self}"/>
       <child link="gimbal_link${self}"/>
-      <origin rpy="0 0 0" xyz="-0.004 0.0 0.0"/>
+      <origin rpy="0 0 0" xyz="0.0 0.0 0.0"/>
       <axis xyz="1 0 0"/>
       <dynamics damping="0.8" friction="0.0"/>
