Commit message: fix urdf and mocap connection

File: robots/crobat/urdf/full_actuated.radxa.gazebo.xacro (robot description, xacro)
@@ -3,5 +3,5 @@
     xmlns:xacro="http://www.ros.org/wiki/xacro" name="crobat" >
   <xacro:arg name="robot_name" default="crobat" />
-  <xacro:include filename="$(find crobat)/urdf/full_actuated.urdf.xacro" />
+  <xacro:include filename="$(find crobat)/urdf/full_actuated.radxa.urdf.xacro" />
   <!-- gazebo plugin for default controller and sensors -->
   <xacro:include filename="$(find aerial_robot_simulation)/xacro/spinal.gazebo.xacro" />

File: robots/crobat/urdf/full_actuated.radxa.urdf.xacro (robot description, xacro)
@@ -3,4 +3,22 @@
     xmlns:xacro="http://www.ros.org/wiki/xacro" name="crobat" >
   <xacro:macro name="crobat_center_link" params="child1 child2 child3 child4">
+    <xacro:macro name="extra_module" params="name parent *origin *inertial visible:=0 model_url:=1 scale:=1">
+      <joint name="${parent}2${name}" type="fixed">
+	<parent link="${parent}"/>
+	<child link="${name}"/>
+	<xacro:insert_block name="origin" />
+      </joint>
+      <link name="${name}">
+	<xacro:insert_block name="inertial" />
+	<xacro:if value="${visible == 1}">
+          <visual>
+            <origin rpy="0 0 0" xyz="0 0 0"/>
+            <geometry>
+              <mesh filename="${model_url}" scale= "${scale} ${scale} ${scale}"/>
+            </geometry>
+          </visual>
+	</xacro:if>
+      </link>
+    </xacro:macro>
     ## dummy
     <link name="root">
@@ -24,5 +42,5 @@
       <inertial>
         <origin xyz="0.0003 -0.0007 0.1399" rpy="0 0 0"/>
-        <mass value="0.0566"/>
+        <mass value="0.0666"/>
         <inertia
             ixx="0.00008943" iyy="0.00008943" izz="0.00006466"
@@ -63,5 +81,5 @@
       <origin xyz="0.0 0 0.103" rpy="${pi/2} 0 0"/>
       <inertial>
-      <mass value = "0.021" />
+      <mass value = "0.023" />
       <origin xyz="0 0 0" rpy="0 0 0"/>
       <inertia
@@ -96,5 +114,5 @@
       <parent link="base_link"/>
       <child link="rotor_arm${child1}"/>
-     <origin rpy="0 0 ${pi/4}" xyz="0.04423 0.04417 0.12801"/>
+      <origin rpy="0 0 ${pi/4}" xyz="0.04423 0.04417 0.12801"/>
       <axis xyz="0 0 1"/>
     </joint>
