Commit message: reverse y-axis and fix urdf

File: robots/crobat/urdf/full_actuated.gazebo.xacro (robot description, xacro)
@@ -3,5 +3,5 @@
     xmlns:xacro="http://www.ros.org/wiki/xacro" name="crobat" >
   <xacro:arg name="robot_name" default="crobat" />
-  <xacro:include filename="$(find crobat)/urdf/full_actuated.urdf.xacro" />
+  <xacro:include filename="$(find crobat)/urdf/full_actuated.serial.urdf.xacro" />
   <!-- gazebo plugin for default controller and sensors -->
   <xacro:include filename="$(find aerial_robot_simulation)/xacro/spinal.gazebo.xacro" />

File: robots/crobat/urdf/full_actuated.serial.urdf.xacro (robot description, xacro)
@@ -1,7 +1,7 @@
 <?xml version="1.0"?>
-<!-- Radxa Cubie A7Z real-machine description. -->
+<!-- Original spinal/rosserial real-machine description. -->
 <robot xmlns:xacro="http://www.ros.org/wiki/xacro" name="crobat">
-  <xacro:arg name="base_mass" default="0.0666" />
-  <xacro:arg name="battery_mass" default="0.023" />
+  <xacro:arg name="base_mass" default="0.0566" />
+  <xacro:arg name="battery_mass" default="0.021" />
   <xacro:include filename="$(find crobat)/urdf/full_actuated.urdf.xacro" />
 </robot>

File: robots/crobat/urdf/full_actuated.urdf.xacro (robot description, xacro)
@@ -2,4 +2,26 @@
 <robot
     xmlns:xacro="http://www.ros.org/wiki/xacro" name="crobat" >
+  <!-- Shared full-actuated geometry. Backend wrappers set only the physical
+       mass values which differ between the spinal and Cubie A7Z assemblies. -->
+  <xacro:arg name="base_mass" default="0.0566" />
+  <xacro:arg name="battery_mass" default="0.021" />
+  <xacro:macro name="extra_module" params="name parent *origin *inertial visible:=0 model_url:=1 scale:=1">
+    <joint name="${parent}2${name}" type="fixed">
+      <parent link="${parent}"/>
+      <child link="${name}"/>
+      <xacro:insert_block name="origin" />
+    </joint>
+    <link name="${name}">
+      <xacro:insert_block name="inertial" />
+      <xacro:if value="${visible == 1}">
+        <visual>
+          <origin rpy="0 0 0" xyz="0 0 0"/>
+          <geometry>
+            <mesh filename="${model_url}" scale="${scale} ${scale} ${scale}"/>
+          </geometry>
+        </visual>
+      </xacro:if>
+    </link>
+  </xacro:macro>
   <xacro:macro name="crobat_center_link" params="child1 child2 child3 child4">
     ## dummy
@@ -24,5 +46,5 @@
       <inertial>
         <origin xyz="0.0003 -0.0007 0.1399" rpy="0 0 0"/>
-        <mass value="0.0566"/>
+        <mass value="$(arg base_mass)"/>
         <inertia
             ixx="0.00008943" iyy="0.00008943" izz="0.00006466"
@@ -63,5 +85,5 @@
       <origin xyz="0.0 0 0.103" rpy="${pi/2} 0 0"/>
       <inertial>
-      <mass value = "0.021" />
+      <mass value="$(arg battery_mass)" />
       <origin xyz="0 0 0" rpy="0 0 0"/>
       <inertia
